File: pcb/pcb/_autosave-pcb.kicad_pcb (KiCad board)
At the start: 2 copper layers, 8 parts, among them J1 Barrel_Jack, J2 Stepper, U1 TSR_1-2433, U2 ESP32-WROOM-32

Commit message: Add esp32
Parts:
- added C3: 100uF, Capacitor_THT:CP_Radial_D5.0mm_P2.50mm, F.Cu at (172.7, 119.4)
Connections:
- A1 pad 2: unconnected-(A1-Pad2) -> +3V3
