File: pcb/pcb/pcb.kicad_sch (KiCad schematic)
At the start: 9 parts, among them J1 Barrel_Jack, J2 Stepper, U1 TSR_1-2433, U2 ESP32-WROOM-32

Commit message: Add esp32
Parts:
- added C1: 1uF, symbol Device:C_Small
- added C2: 10uF, symbol Device:C_Small
- added C3: 0.1uF, symbol Device:C_Small
- added J1: UART, Connector_PinHeader_2.54mm:PinHeader_1x03_P2.54mm_Vertical, symbol Connector_Generic:Conn_01x03
- added R1: 10k, symbol Device:R
- renumbered C3 to C4, C1 to C5, C2 to C6, J1 to J2, J2 to J3, U2 to U1, U1 to U2
Connections:
- net +3V3: now also U1.2 (VDD), C2.1, C3.1, R1.1
- net GND: now also U1.1 (GND), U1.15 (GND), U1.38 (GND), U1.39 (GND), C1.2, C2.2, C3.2, J1.3 (Pin_3)
- net RX: now reaches U1.24 (IO2)
- net RX: now also J1.2 (Pin_2)
- net at U1.3 (EN): now also C1.1, R1.2
- net TX: now reaches U1.35 (TXD0/IO1)
- net TX: now also J1.1 (Pin_1)
- net DIR: now reaches U1.6 (IO34)
- net DIR: now also A1.16 (DIR)
- net SLP: now reaches U1.7 (IO35)
- net SLP: now also A1.14 (~{SLP})
- net STEP: now reaches U1.9 (IO33)
- net STEP: now also A1.15 (STEP)
Other:
- note added: "ESP32"
- moved on the sheet: U1

Commit message: basic pcb layout
Parts:
- C1, C2, C3: footprint (none) -> Capacitor_SMD:C_1206_3216Metric_Pad1.33x1.80mm_HandSolder
- R1: footprint (none) -> Resistor_SMD:R_1206_3216Metric_Pad1.30x1.75mm_HandSolder
Changed lines of the file:
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@@
     (property "Reference" "C1" (id 0) (at 34.29 90.17 90))
     (property "Value" "1uF" (id 1) (at 34.29 95.25 90))
-    (property "Footprint" "" (id 2) (at 34.29 92.71 0)
+    (property "Footprint" "Capacitor_SMD:C_1206_3216Metric_Pad1.33x1.80mm_HandSolder" (id 2) (at 34.29 92.71 0)
       (effects (font (size 1.27 1.27)) hide)
     )
@@
       (effects (font (size 1.27 1.27)) (justify left))
     )
-    (property "Footprint" "" (id 2) (at 38.862 87.63 90)
+    (property "Footprint" "Resistor_SMD:R_1206_3216Metric_Pad1.30x1.75mm_HandSolder" (id 2) (at 38.862 87.63 90)
       (effects (font (size 1.27 1.27)) hide)
     )
@@
       (effects (font (size 1.27 1.27)) (justify left))
     )
-    (property "Footprint" "" (id 2) (at 52.07 67.31 0)
+    (property "Footprint" "Capacitor_SMD:C_1206_3216Metric_Pad1.33x1.80mm_HandSolder" (id 2) (at 52.07 67.31 0)
       (effects (font (size 1.27 1.27)) hide)
     )
@@
       (effects (font (size 1.27 1.27)) (justify left))
     )
-    (property "Footprint" "" (id 2) (at 39.37 67.31 0)
+    (property "Footprint" "Capacitor_SMD:C_1206_3216Metric_Pad1.33x1.80mm_HandSolder" (id 2) (at 39.37 67.31 0)
       (effects (font (size 1.27 1.27)) hide)
     )
@@
     )
     (path "/5b053de1-d132-4184-809e-d854fad21bc8"
-      (reference "C1") (unit 1) (value "1uF") (footprint "")
+      (reference "C1") (unit 1) (value "1uF") (footprint "Capacitor_SMD:C_1206_3216Metric_Pad1.33x1.80mm_HandSolder")
     )
     (path "/b989eb92-f813-477a-809c-6e6478d4521b"
-      (reference "C2") (unit 1) (value "10uF") (footprint "")
+      (reference "C2") (unit 1) (value "10uF") (footprint "Capacitor_SMD:C_1206_3216Metric_Pad1.33x1.80mm_HandSolder")
     )
     (path "/9a0b6919-48cc-44cf-b0ea-1c0f31d6f58a"
-      (reference "C3") (unit 1) (value "0.1uF") (footprint "")
+      (reference "C3") (unit 1) (value "0.1uF") (footprint "Capacitor_SMD:C_1206_3216Metric_Pad1.33x1.80mm_HandSolder")
     )
     (path "/b698d2dc-df41-461d-8031-8b8ce841d1ca"
@@
     )
     (path "/618b85b8-3878-4dca-95c1-d1249ea332c0"
-      (reference "R1") (unit 1) (value "10k ") (footprint "")
+      (reference "R1") (unit 1) (value "10k ") (footprint "Resistor_SMD:R_1206_3216Metric_Pad1.30x1.75mm_HandSolder")
     )
     (path "/66f41d59-e5a3-4e8f-8f6c-d365e8eefce7"

Commit message: Route pcb
Parts:
- added H1: MountingHole, MountingHole:MountingHole_2.7mm_M2.5_Pad, symbol Mechanical:MountingHole
- added H2, H3, H4: MountingHole, MountingHole:MountingHole_2.5mm_Pad, symbol Mechanical:MountingHole
Changed lines of the file:
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@@
     (effects (font (size 1.27 1.27)) (justify left bottom))
+  )
+  (symbol (lib_id "Mechanical:MountingHole") (at 52.07 27.94 0) (unit 1)
+    (in_bom yes) (on_board yes) (fields_autoplaced)
+    (property "Reference" "H2" (id 0) (at 54.61 26.6699 0)
+      (effects (font (size 1.27 1.27)) (justify left))
+    )
+    (property "Value" "MountingHole" (id 1) (at 54.61 29.2099 0)
+      (effects (font (size 1.27 1.27)) (justify left))
+    )
+    (property "Footprint" "MountingHole:MountingHole_2.5mm_Pad" (id 2) (at 52.07 27.94 0)
+      (effects (font (size 1.27 1.27)) hide)
+    )
+    (property "Datasheet" "~" (id 3) (at 52.07 27.94 0)
+      (effects (font (size 1.27 1.27)) hide)
+    )
   )
   (symbol (lib_id "power:GND") (at 213.36 68.58 270) (unit 1)
@@
     (pin "1")
     (pin "2")
+  )
+  (symbol (lib_id "Mechanical:MountingHole") (at 34.29 27.94 0) (unit 1)
+    (in_bom yes) (on_board yes) (fields_autoplaced)
+    (property "Reference" "H1" (id 0) (at 36.83 26.6699 0)
+      (effects (font (size 1.27 1.27)) (justify left))
+    )
+    (property "Value" "MountingHole" (id 1) (at 36.83 29.2099 0)
+      (effects (font (size 1.27 1.27)) (justify left))
+    )
+    (property "Footprint" "MountingHole:MountingHole_2.7mm_M2.5_Pad" (id 2) (at 34.29 27.94 0)
+      (effects (font (size 1.27 1.27)) hide)
+    )
+    (property "Datasheet" "~" (id 3) (at 34.29 27.94 0)
+      (effects (font (size 1.27 1.27)) hide)
+    )
   )
   (symbol (lib_id "Device:C") (at 226.06 64.77 0) (unit 1)
@@
     (pin "9")
   )
+  (symbol (lib_id "Mechanical:MountingHole") (at 69.85 27.94 0) (unit 1)
+    (in_bom yes) (on_board yes) (fields_autoplaced)
+    (property "Reference" "H3" (id 0) (at 72.39 26.6699 0)
+      (effects (font (size 1.27 1.27)) (justify left))
+    )
+    (property "Value" "MountingHole" (id 1) (at 72.39 29.2099 0)
+      (effects (font (size 1.27 1.27)) (justify left))
+    )
+    (property "Footprint" "MountingHole:MountingHole_2.5mm_Pad" (id 2) (at 69.85 27.94 0)
+      (effects (font (size 1.27 1.27)) hide)
+    )
+    (property "Datasheet" "~" (id 3) (at 69.85 27.94 0)
+      (effects (font (size 1.27 1.27)) hide)
+    )
+  )
   (symbol (lib_id "power:GND") (at 109.22 92.71 0) (unit 1)
     (in_bom yes) (on_board yes) (fields_autoplaced)
@@
     (pin "1")
   )
+  (symbol (lib_id "Mechanical:MountingHole") (at 87.63 27.94 0) (unit 1)
+    (in_bom yes) (on_board yes) (fields_autoplaced)
+    (property "Reference" "H4" (id 0) (at 90.17 26.6699 0)
+      (effects (font (size 1.27 1.27)) (justify left))
+    )
+    (property "Value" "MountingHole" (id 1) (at 90.17 29.2099 0)
+      (effects (font (size 1.27 1.27)) (justify left))
+    )
+    (property "Footprint" "MountingHole:MountingHole_2.5mm_Pad" (id 2) (at 87.63 27.94 0)
+      (effects (font (size 1.27 1.27)) hide)
+    )
+    (property "Datasheet" "~" (id 3) (at 87.63 27.94 0)
+      (effects (font (size 1.27 1.27)) hide)
+    )
+  )
   (symbol (lib_id "power:GND") (at 31.75 92.71 270) (unit 1)
     (in_bom yes) (on_board yes) (fields_autoplaced)
@@
       (reference "C6") (unit 1) (value "10uF") (footprint "Capacitor_SMD:C_1206_3216Metric_Pad1.33x1.80mm_HandSolder")
     )
+    (path "/34fa3d54-c535-425c-b022-e1943d8d5f86"
+      (reference "H1") (unit 1) (value "MountingHole") (footprint "MountingHole:MountingHole_2.7mm_M2.5_Pad")
+    )
+    (path "/00d9b647-6f7b-4061-b8f8-f07282eb45d6"
+      (reference "H2") (unit 1) (value "MountingHole") (footprint "MountingHole:MountingHole_2.5mm_Pad")
+    )
+    (path "/72d1a3aa-0e7b-4b10-a84c-7a0d93e80db5"
+      (reference "H3") (unit 1) (value "MountingHole") (footprint "MountingHole:MountingHole_2.5mm_Pad")
+    )
+    (path "/b3ffd185-6873-4234-b901-27672efba3ad"
+      (reference "H4") (unit 1) (value "MountingHole") (footprint "MountingHole:MountingHole_2.5mm_Pad")
+    )
     (path "/f859e7d0-40bd-4ce3-9e1e-50d116474f0f"
